Commit message: 适配 LiDAR 45° 前倾安装：TF、CropBox、Costmap 参数
- TF 变换 base_link→livox_frame: pitch 0→0.7854 (45°)，覆盖真机+仿真共7个文件
- CropBox 参数适配 livox_frame 坐标系下的 45° 倾斜车体投影
- Costmap 调优: observation_persistence=0.6, clear_after_reading=false, voxel_min_points=2, mark_threshold=1
- 移除未连接 RealSense 相机的启动和 costmap 残留引用
- filter_node: 清理未使用的 voxel_grid 代码，修正 CropBox 可视化标记帧

Co-Authored-By: Claude Opus 4.7 (1M context) <noreply@anthropic.com>

File: cod_-rm2026_-navigation-master/src/cod_gazebo_simulator/resource/cod_robot.urdf.xacro (robot description, xacro)
@@ -68,5 +68,5 @@
     <parent link="base_link"/>
     <child link="livox_frame"/>
-    <origin xyz="0.0 0.0 0.15" rpy="0 0 0"/>
+    <origin xyz="0.0 0.0 0.15" rpy="0 0.7854 0"/>   <!-- Pitch +45°: LiDAR前倾 -->
   </joint>
   <!-- ===== Gazebo 差速驱动插件 (sub cmd_vel → apply wheel velocity) ===== -->
